File: hardware/Microgrid-Home-Energy-Monitor.kicad_sch (KiCad schematic)
At the start: 32 parts, among them J1 AudioJack2, J2 AudioJack2, J3 Conn_01x04, J4 USB_C_Receptacle_USB2.0_16P, J5 Conn_01x06, J6 Conn_01x03, SW1 SW_Push, SW2 SW_Push, U1 ESP32-WROOM-32, U2 MCP6002-xP, U3 AMS1117-3.3

Commit message: Fix all DRC errors; sync fixed board + fresh Gerbers into repo
Board fixes (done in KiCad GUI):
- Added solid GND plane on B.Cu; stitching vias tie front pour fragments
  to it -- eliminates the split-pour GND islands permanently
- ESP32 thermal vias: 0.2mm -> 0.3mm drill (JLCPCB 2-layer minimum)
- Min clearance relaxed to fit the USB-C (J4) footprint's 0.15mm pad gaps

Verified with kicad-cli: DRC 0 violations, 0 unconnected. ERC 0 errors.
Gerbers + drill files re-exported from the fixed board -- ready for JLCPCB.

Note: the repo previously carried a stale June 14 copy of the board; the
edited project lived outside the repo. This commit syncs the real files.

Co-Authored-By: Claude Fable 5 <noreply@anthropic.com>
Parts:
- added D1, D2: LED, LED_THT:LED_D3.0mm, symbol Device:LED
- added R13, R14: 150, Resistor_SMD:R_0603_1608Metric, symbol Device:R
- added TP1, TP2, TP3, TP4, TP5: TestPoint, TestPoint:TestPoint_Pad_D1.5mm, symbol Connector:TestPoint
- C1, C2, C3, C6, C8: footprint (none) -> Capacitor_SMD:C_0805_2012Metric
- C4, C5, C7, C9: footprint (none) -> Capacitor_SMD:C_0603_1608Metric
- J1, J2: footprint (none) -> Connector_Audio:Jack_3.5mm_CUI_SJ-3523-SMT_Horizontal
- J3: footprint (none) -> Connector_PinHeader_2.54mm:PinHeader_1x04_P2.54mm_Vertical
- J4: footprint (none) -> Connector_USB:USB_C_Receptacle_GCT_USB4085
- J5: footprint (none) -> Connector_PinHeader_2.54mm:PinHeader_1x06_P2.54mm_Vertical
- J6: footprint (none) -> Connector_PinHeader_2.54mm:PinHeader_1x03_P2.54mm_Vertical
- R1, R10, R11, R12, R2, R3, R4, R5, R6, R7, R8, R9: footprint (none) -> Resistor_SMD:R_0603_1608Metric
- SW1, SW2: footprint (none) -> Button_Switch_THT:SW_PUSH_6mm_H4.3mm
- U2: footprint (none) -> Package_DIP:DIP-8_W7.62mm
Connections:
- net +3.3V: now also R13.1, TP2.1
- net EN: now also TP4.1
- net GND: now also D1.1 (K), D2.1 (K), TP3.1
- net IO0: now also TP5.1
- net VBUS: now also TP1.1
- net at U1.24 (IO2): now also R14.1
- new net: D2.2 (A), R14.2
- new net: D1.2 (A), R13.2
- no-connect marks 31 -> 30
